Commit message: feat: Apply booster_assets for GMR

File: assets/booster_t1/T1_29dof.urdf (robot description, URDF)
Before this commit: robot T1, 24 links, 23 joints
Links:
- added link AL4, mass 0.5570; collision cylinder length=0.14 radius=0.04; visual mesh filename=meshes/AL4.STL
- added link AL5, mass 0.43402; visual mesh filename=meshes/AL5.STL
- added link AL6, mass 0.47922; visual mesh filename=meshes/AL6.STL
- added link AR4, mass 0.5570; collision cylinder length=0.14 radius=0.04; visual mesh filename=meshes/AR4.STL
- added link AR5, mass 0.43402; visual mesh filename=meshes/AR5.STL
- added link AR6, mass 0.47922; visual mesh filename=meshes/AR6.STL
- link AL1: geometry collision cylinder length=0.07 radius=0.03; visual mesh filename=meshes/AL1.STL
- link AL3: geometry collision cylinder length=0.19 radius=0.03; visual mesh filename=meshes/AL3.STL
- link AR1: geometry collision cylinder length=0.07 radius=0.03; visual mesh filename=meshes/AR1.STL
- link AR3: geometry collision cylinder length=0.19 radius=0.03; visual mesh filename=meshes/AR3.STL
- link H1: geometry collision cylinder length=0.07 radius=0.025; visual mesh filename=meshes/H1.STL
- link Hip_Pitch_Left: geometry collision cylinder length=0.085 radius=0.045; visual mesh filename=meshes/Hip_Pitch_Left.STL
- link Hip_Pitch_Right: geometry collision cylinder length=0.085 radius=0.045; visual mesh filename=meshes/Hip_Pitch_Right.STL
- link Hip_Roll_Left: geometry collision cylinder length=0.08 radius=0.045; visual mesh filename=meshes/Hip_Roll_Left.STL
- link Hip_Roll_Right: geometry collision cylinder length=0.08 radius=0.045; visual mesh filename=meshes/Hip_Roll_Right.STL
- link Hip_Yaw_Left: geometry collision cylinder length=0.09 radius=0.055; visual mesh filename=meshes/Hip_Yaw_Left.STL
- link Hip_Yaw_Right: geometry collision cylinder length=0.09 radius=0.055; visual mesh filename=meshes/Hip_Yaw_Right.STL
- link Shank_Left: mass 1.73 -> 1.82; geometry collision box size=0.1 0.08 0.14; visual mesh filename=meshes/Shank_Left.STL
- link Shank_Right: mass 1.79 -> 1.82; geometry collision box size=0.1 0.08 0.14; visual mesh filename=meshes/Shank_Right.STL
- link Trunk: geometry collision box size=0.17 0.18 0.29; visual mesh filename=meshes/Logo.STL
- link Waist: geometry collision cylinder length=0.1 radius=0.06; visual mesh filename=meshes/Waist.STL
- link left_foot_link: geometry collision box size=0.224868 0.1 0.04366; visual mesh filename=meshes/left_foot_link.STL
- link left_hand_link: mass 0.327214390850251 -> 0.30603; geometry collision cylinder length=0.15 radius=0.06; visual mesh filename=meshes/AL7.STL
- link right_foot_link: geometry collision box size=0.224868 0.1 0.04366; visual mesh filename=meshes/right_foot_link.STL
- link right_hand_link: mass 0.327214390850251 -> 0.30603; geometry collision cylinder length=0.15 radius=0.06; visual mesh filename=meshes/AR7.STL
Joints:
- added joint Left_Hand_Roll: type revolute, parent AL6, child left_hand_link, origin xyz=0.00475 0.07 0.0015 rpy=0 0 0, axis 1 0 0, limit lower=-0.758 upper=1.4285 effort=7 velocity=12.56
- added joint Left_Wrist_Pitch: type revolute, parent AL4, child AL5, origin xyz=0 0.105 0.00025 rpy=0 0 0, axis 0 1 0, limit lower=-2.5821 upper=2.5821 effort=7 velocity=12.56
- added joint Left_Wrist_Yaw: type revolute, parent AL5, child AL6, origin xyz=0 0.042 0 rpy=0 0 0, axis 0 0 1, limit lower=-1.8185 upper=1.4261 effort=18 velocity=18
- added joint Right_Hand_Roll: type revolute, parent AR6, child right_hand_link, origin xyz=0.00475 -0.07 0.0015 rpy=0 0 0, axis 1 0 0, limit lower=-1.4285 upper=0.758 effort=7 velocity=12.56
- added joint Right_Wrist_Pitch: type revolute, parent AR4, child AR5, origin xyz=0 -0.105 0.00025 rpy=0 0 0, axis 0 1 0, limit lower=-2.5821 upper=2.5821 effort=7 velocity=12.56
- added joint Right_Wrist_Yaw: type revolute, parent AR5, child AR6, origin xyz=0 -0.042 0 rpy=0 0 0, axis 0 0 1, limit lower=-1.4261 upper=1.8185 effort=18 velocity=18
- joint AAHead_yaw: limit lower=-1.57 upper=1.57 effort=7 velocity=12.56 -> lower=-1.0472 upper=1.0472 effort=7 velocity=12.56
- joint Head_pitch: limit lower=-0.35 upper=1.22 effort=7 velocity=12.56 -> lower=-0.3491 upper=0.8552 effort=7 velocity=12.56
- joint Left_Ankle_Pitch: limit lower=-0.87 upper=0.35 effort=20 velocity=18.8 -> lower=-0.87 upper=0.35 effort=24 velocity=12.9
- joint Left_Ankle_Roll: limit lower=-0.44 upper=0.44 effort=15 velocity=12.4 -> lower=-0.44 upper=0.44 effort=15 velocity=12.9
- joint Left_Elbow_Pitch: limit lower=-2.27 upper=2.27 effort=18 velocity=18.84 -> lower=-2.234 upper=2.234 effort=18 velocity=18
- joint Left_Elbow_Yaw: child left_hand_link -> AL4; limit lower=-2.44 upper=0 effort=18 velocity=18.84 -> lower=-2.1402 upper=1.6844 effort=18 velocity=18
- joint Left_Hip_Pitch: limit lower=-1.8 upper=1.57 effort=45 velocity=12.5 -> lower=-3.0020 upper=2.2166 effort=45 velocity=15.2
- joint Left_Hip_Roll: limit lower=-0.2 upper=1.57 effort=30 velocity=10.9 -> lower=-0.2 upper=1.57 effort=25 velocity=7.1
- joint Left_Hip_Yaw: limit lower=-1 upper=1 effort=30 velocity=10.9 -> lower=-1 upper=1 effort=25 velocity=7.1
- joint Left_Knee_Pitch: limit lower=0 upper=2.34 effort=60 velocity=11.7 -> lower=0 upper=2.1817 effort=60 velocity=14.7
- joint Left_Shoulder_Pitch: limit lower=-3.31 upper=1.22 effort=18 velocity=18.84 -> lower=-3.29 upper=1.18 effort=18 velocity=18
- joint Left_Shoulder_Roll: limit lower=-1.74 upper=1.57 effort=18 velocity=18.84 -> lower=-1.577 upper=1.7055 effort=18 velocity=18
- joint Right_Ankle_Pitch: limit lower=-0.87 upper=0.35 effort=20 velocity=18.8 -> lower=-0.87 upper=0.35 effort=24 velocity=12.9
- joint Right_Ankle_Roll: limit lower=-0.44 upper=0.44 effort=15 velocity=12.4 -> lower=-0.44 upper=0.44 effort=15 velocity=12.9
- joint Right_Elbow_Pitch: limit lower=-2.27 upper=2.27 effort=18 velocity=18.84 -> lower=-2.234 upper=2.234 effort=18 velocity=18
- joint Right_Elbow_Yaw: child right_hand_link -> AR4; limit lower=0 upper=2.44 effort=18 velocity=18.84 -> lower=-1.6844 upper=2.1402 effort=18 velocity=18
- joint Right_Hip_Pitch: limit lower=-1.8 upper=1.57 effort=45 velocity=12.5 -> lower=-3.0020 upper=2.2166 effort=45 velocity=15.2
- joint Right_Hip_Roll: limit lower=-1.57 upper=0.2 effort=30 velocity=10.9 -> lower=-1.57 upper=0.2 effort=25 velocity=7.1
- joint Right_Hip_Yaw: limit lower=-1 upper=1 effort=30 velocity=10.9 -> lower=-1 upper=1 effort=25 velocity=7.1
- joint Right_Knee_Pitch: limit lower=0 upper=2.34 effort=60 velocity=11.7 -> lower=0 upper=2.1817 effort=60 velocity=14.7
- joint Right_Shoulder_Pitch: limit lower=-3.31 upper=1.22 effort=18 velocity=18.84 -> lower=-3.29 upper=1.1868 effort=18 velocity=18
- joint Right_Shoulder_Roll: limit lower=-1.57 upper=1.74 effort=18 velocity=18.84 -> lower=-1.7055 upper=1.577 effort=18 velocity=18
- joint Waist: limit lower=-1.57 upper=1.57 effort=30 velocity=10.88 -> lower=-1.57 upper=1.57 effort=25 velocity=7.1

File: assets/booster_t1/T1_locomotion.urdf (robot description, URDF)
Before this commit: robot T1, 24 links, 23 joints
Links:
- link AL1: geometry collision cylinder length=0.07 radius=0.03; visual mesh filename=meshes/AL1.STL
- link AL3: geometry collision cylinder length=0.19 radius=0.03; visual mesh filename=meshes/AL3.STL
- link AR1: geometry collision cylinder length=0.07 radius=0.03; visual mesh filename=meshes/AR1.STL
- link AR3: geometry collision cylinder length=0.19 radius=0.03; visual mesh filename=meshes/AR3.STL
- link H1: geometry collision cylinder length=0.07 radius=0.025; visual mesh filename=meshes/H1.STL
- link H2: geometry collision sphere radius=0.08; visual mesh filename=meshes/H2.STL
- link Hip_Pitch_Left: geometry collision cylinder length=0.085 radius=0.045; visual mesh filename=meshes/Hip_Pitch_Left.STL
- link Hip_Pitch_Right: geometry collision cylinder length=0.085 radius=0.045; visual mesh filename=meshes/Hip_Pitch_Right.STL
- link Hip_Roll_Left: geometry collision cylinder length=0.08 radius=0.045; visual mesh filename=meshes/Hip_Roll_Left.STL
- link Hip_Roll_Right: geometry collision cylinder length=0.08 radius=0.045; visual mesh filename=meshes/Hip_Roll_Right.STL
- link Hip_Yaw_Left: geometry collision cylinder length=0.09 radius=0.055; visual mesh filename=meshes/Hip_Yaw_Left.STL
- link Hip_Yaw_Right: geometry collision cylinder length=0.09 radius=0.055; visual mesh filename=meshes/Hip_Yaw_Right.STL
- link Shank_Left: mass 1.73 -> 1.82; geometry collision box size=0.1 0.08 0.14; visual mesh filename=meshes/Shank_Left.STL
- link Shank_Right: mass 1.79 -> 1.82; geometry collision box size=0.1 0.08 0.14; visual mesh filename=meshes/Shank_Right.STL
- link Trunk: geometry collision box size=0.17 0.18 0.29; visual mesh filename=meshes/Logo.STL
- link Waist: geometry collision cylinder length=0.1 radius=0.06; visual mesh filename=meshes/Waist.STL
- link left_foot_link: geometry collision box size=0.224868 0.1 0.04366; visual mesh filename=meshes/left_foot_link.STL
- link left_hand_link: geometry collision cylinder length=0.13 radius=0.029; visual mesh filename=meshes/left_hand_link.STL
- link right_foot_link: geometry collision box size=0.224868 0.1 0.04366; visual mesh filename=meshes/right_foot_link.STL
- link right_hand_link: geometry collision cylinder length=0.13 radius=0.029; visual mesh filename=meshes/right_hand_link.STL
Joints:
- joint AAHead_yaw: limit lower=-1.57 upper=1.57 effort=7 velocity=12.56 -> lower=-1.0472 upper=1.0472 effort=7 velocity=12.56
- joint Head_pitch: limit lower=-0.35 upper=1.22 effort=7 velocity=12.56 -> lower=-0.3491 upper=0.8552 effort=7 velocity=12.56
- joint Left_Ankle_Pitch: limit lower=-0.87 upper=0.35 effort=24 velocity=18.8 -> lower=-0.87 upper=0.35 effort=24 velocity=12.9
- joint Left_Ankle_Roll: limit lower=-0.44 upper=0.44 effort=15 velocity=12.4 -> lower=-0.44 upper=0.44 effort=15 velocity=12.9
- joint Left_Elbow_Pitch: limit lower=-2.27 upper=2.27 effort=18 velocity=18.84 -> lower=-2.234 upper=2.234 effort=18 velocity=18
- joint Left_Elbow_Yaw: limit lower=-2.44 upper=0 effort=18 velocity=18.84 -> lower=-2.1402 upper=1.6844 effort=18 velocity=18; origin xyz=0 0.1471 0 rpy=0 0 -0.5 -> xyz=0 0.1471 0 rpy=0 0 0
- joint Left_Hip_Pitch: limit lower=-1.8 upper=1.57 effort=45 velocity=12.5 -> lower=-3.0020 upper=2.2166 effort=45 velocity=15.2
- joint Left_Hip_Roll: limit lower=-0.3 upper=1.57 effort=30 velocity=10.9 -> lower=-0.2 upper=1.57 effort=25 velocity=7.1
- joint Left_Hip_Yaw: limit lower=-1 upper=1 effort=30 velocity=10.9 -> lower=-1 upper=1 effort=25 velocity=7.1
- joint Left_Knee_Pitch: limit lower=0 upper=2.34 effort=60 velocity=11.7 -> lower=0 upper=2.1817 effort=60 velocity=14.7
- joint Left_Shoulder_Pitch: limit lower=-3.31 upper=1.22 effort=18 velocity=18.84 -> lower=-3.29 upper=1.18 effort=18 velocity=18; origin xyz=0.0575 0.1063 0.219 rpy=0 0.2 0 -> xyz=0.0575 0.1063 0.219 rpy=0 0.00088113 0
- joint Left_Shoulder_Roll: limit lower=-1.74 upper=1.57 effort=18 velocity=18.84 -> lower=-1.577 upper=1.7055 effort=18 velocity=18; origin xyz=0 0.047 0 rpy=-1.35 0 0 -> xyz=0 0.047 0 rpy=0 0 0
- joint Right_Ankle_Pitch: limit lower=-0.87 upper=0.35 effort=24 velocity=18.8 -> lower=-0.87 upper=0.35 effort=24 velocity=12.9
- joint Right_Ankle_Roll: limit lower=-0.44 upper=0.44 effort=15 velocity=12.4 -> lower=-0.44 upper=0.44 effort=15 velocity=12.9
- joint Right_Elbow_Pitch: limit lower=-2.27 upper=2.27 effort=18 velocity=18.84 -> lower=-2.234 upper=2.234 effort=18 velocity=18
- joint Right_Elbow_Yaw: limit lower=0 upper=2.44 effort=18 velocity=18.84 -> lower=-1.6844 upper=2.1402 effort=18 velocity=18; origin xyz=0 -0.1471 0 rpy=0 0 0.5 -> xyz=0 -0.1471 0 rpy=0 0 0
- joint Right_Hip_Pitch: limit lower=-1.8 upper=1.57 effort=45 velocity=12.5 -> lower=-3.0020 upper=2.2166 effort=45 velocity=15.2
- joint Right_Hip_Roll: limit lower=-1.57 upper=0.3 effort=30 velocity=10.9 -> lower=-1.57 upper=0.2 effort=25 velocity=7.1
- joint Right_Hip_Yaw: limit lower=-1 upper=1 effort=30 velocity=10.9 -> lower=-1 upper=1 effort=25 velocity=7.1
- joint Right_Knee_Pitch: limit lower=0 upper=2.34 effort=60 velocity=11.7 -> lower=0 upper=2.1817 effort=60 velocity=14.7
- joint Right_Shoulder_Pitch: limit lower=-3.31 upper=1.22 effort=18 velocity=18.84 -> lower=-3.29 upper=1.1868 effort=18 velocity=18; origin xyz=0.0575 -0.1063 0.219 rpy=0 0.2 0 -> xyz=0.0575 -0.1063 0.219 rpy=0 0.00088113 0
- joint Right_Shoulder_Roll: limit lower=-1.57 upper=1.74 effort=18 velocity=18.84 -> lower=-1.7055 upper=1.577 effort=18 velocity=18; origin xyz=0 -0.047 0 rpy=1.35 0 0 -> xyz=0 -0.047 0 rpy=0 0 0
- joint Waist: limit lower=-1.57 upper=1.57 effort=30 velocity=10.88 -> lower=-1.57 upper=1.57 effort=25 velocity=7.1
